Commit message: completed robot URDF

File: src/arduinobot_description/urdf/arduinobot.urdf.xacro (robot description, xacro)
@@ -21,5 +21,5 @@
     <link name="base_plate">
         <visual>
-            <origin rpy="-0 0 0" xyz="-0.39 -0.39 -0.56" />
+            <origin rpy="0 0 0" xyz="-0.39 -0.39 -0.56" />
             <geometry>
                 <mesh filename="package://arduinobot_description/meshes/base_plate.STL"
@@ -31,7 +31,86 @@
         <parent link="base_link" />
         <child link="base_plate" />
-        <axis xyz="0 0 1"/>
+        <axis xyz="0 0 1" />
         <origin rpy="0 0 0" xyz="0 0 0.307" />
         <limit lower="-${PI/2}" upper="${PI/2}" effort="${effort}" velocity="${velocity}" />
     </joint>
+    <link name="forward_drive_arm">
+        <visual>
+            <origin rpy="0 -${PI/2} ${PI/2}" xyz="0.19 0.06 -0.08" />
+            <geometry>
+                <mesh filename="package://arduinobot_description/meshes/forward_drive_arm.STL"
+                    scale="0.01 0.01 0.01" />
+            </geometry>
+        </visual>
+    </link>
+    <joint name="joint_2" type="revolute">
+        <parent link="base_plate" />
+        <child link="forward_drive_arm" />
+        <axis xyz="1 0 0" />
+        <origin rpy="0 0 0" xyz="-0.02 0 0.35" />
+        <limit lower="-${PI/2}" upper="${PI/2}" effort="${effort}" velocity="${velocity}" />
+    </joint>
+    <link name="horizontal_arm">
+        <visual>
+            <origin rpy="${PI/2} 0 ${PI/2}" xyz="-0.03 -0.4 -0.06" />
+            <geometry>
+                <mesh filename="package://arduinobot_description/meshes/horizontal_arm.STL"
+                    scale="0.01 0.01 0.01" />
+            </geometry>
+        </visual>
+    </link>
+    <joint name="joint_3" type="revolute">
+        <parent link="forward_drive_arm" />
+        <child link="horizontal_arm" />
+        <axis xyz="1 0 0" />
+        <origin rpy="0 0 0" xyz="0 0 0.8" />
+        <limit lower="-${PI/2}" upper="${PI/2}" effort="${effort}" velocity="${velocity}" />
+    </joint>
+    <link name="claw_support">
+        <visual>
+            <origin rpy="0 0 ${PI/2}" xyz="0.13 -0.05 -0.15" />
+            <geometry>
+                <mesh filename="package://arduinobot_description/meshes/claw_support.STL"
+                    scale="0.01 0.01 0.01" />
+            </geometry>
+        </visual>
+    </link>
+    <joint name="horizontal_arm_to_claw_support" type="fixed">
+        <parent link="horizontal_arm" />
+        <child link="claw_support" />
+        <origin rpy="0 0 0" xyz="0 0.82 0" />
+    </joint>
+    <link name="gripper_right">
+        <visual>
+            <origin rpy="0 0 -${PI/2}" xyz="-0.09 0.48 -0.08" />
+            <geometry>
+                <mesh filename="package://arduinobot_description/meshes/right_finger.STL"
+                    scale="0.01 0.01 0.01" />
+            </geometry>
+        </visual>
+    </link>
+    <link name="gripper_left">
+        <visual>
+            <origin rpy="0 0 -${PI/2}" xyz="-0.03 0.48 -0.08" />
+            <geometry>
+                <mesh filename="package://arduinobot_description/meshes/left_finger.STL"
+                    scale="0.01 0.01 0.01" />
+            </geometry>
+        </visual>
+    </link>
+    <joint name="joint_4" type="revolute">
+        <parent link="claw_support" />
+        <child link="gripper_right" />
+        <axis xyz="0 0 1" />
+        <origin rpy="0 0 0" xyz="0.09 0.15 -0.1" />
+        <limit lower="-${PI/2}" upper="0" effort="${effort}" velocity="${velocity}" />
+    </joint>
+    <joint name="joint_5" type="revolute">
+        <parent link="claw_support" />
+        <child link="gripper_left" />
+        <axis xyz="0 0 1" />
+        <origin rpy="0 0 0" xyz="-0.09 0.15 -0.1" />
+        <limit lower="0" upper="${PI/2}" effort="${effort}" velocity="${velocity}" />
+        <mimic joint="joint_4" multiplier="-1" />
+    </joint>
 </robot>

Commit message: gazebo launch file

File: src/arduinobot_description/urdf/arduinobot.urdf.xacro (robot description, xacro)
@@ -4,6 +4,15 @@
     <xacro:property name="effort" value="30.0" />
     <xacro:property name="velocity" value="10.0" />
+    <xacro:macro name="default_inertial" params="mass">
+        <inertial>
+            <mass value="${mass}" />
+            <inertia ixx="1.0" ixy="0.0" ixz="0.0"
+                iyy="1.0" iyz="0.0"
+                izz="1.0" />
+        </inertial>
+    </xacro:macro>
     <link name="world" />
     <link name="base_link">
+        <xacro:default_inertial mass="1.0" />
         <visual>
             <origin rpy="0 0 0" xyz="-0.5 -0.5 0" />
@@ -12,5 +21,13 @@
                     scale="0.01 0.01 0.01" />
             </geometry>
-        </visual>
+            <material name="red"/>
+        </visual>
+        <collision>
+            <origin rpy="0 0 0" xyz="-0.5 -0.5 0" />
+            <geometry>
+                <mesh filename="package://arduinobot_description/meshes/basement.STL"
+                    scale="0.01 0.01 0.01" />
+            </geometry>
+        </collision>
     </link>
     <joint name="virtual_joint" type="fixed">
@@ -19,5 +36,76 @@
         <origin rpy="0 0 0" xyz="0 0 0" />
     </joint>
+    <link name="rgb_camera ">
+        <xacro:default_inertial mass="0.01" />
+        <visual>
+            <origin rpy="${2*PI/3} ${PI} ${PI}" xyz="-0.127 0.35 0.3" />
+            <geometry>
+                <mesh filename="package://arduinobot_description/meshes/pi_camera.STL"
+                    scale="0.01 0.01 0.01" />
+            </geometry>
+            <material name="blue"/>
+        </visual>
+        <collision>
+            <origin rpy="${2*PI/3} ${PI} ${PI}" xyz="-0.127 0.35 0.3" />
+            <geometry>
+                <mesh filename="package://arduinobot_description/meshes/pi_camera.STL"
+                    scale="0.01 0.01 0.01" />
+            </geometry>
+        </collision>
+    </link>
+    <gazebo reference="rgb_camera">
+        <sensor type="camera" name="rgb_camera_sensor">
+            <update_rate>30.0</update_rate>
+            <always_on>true</always_on>
+            <vizualize>true</vizualize>
+            <!-- <gz_frame_id>/rgb_camera</gz_frame_id> -->
+            <camera name="rgb_camera">
+                <horizontal_fov>1.15</horizontal_fov>
+                <vertical_fov>0.71</vertical_fov>
+                <image>
+                    <width>2304</width>
+                    <height>1296</height>
+                    <format>R8G8B8</format>
+                </image>
+                <distortion>
+                    <k1>0.0</k1>
+                    <k2>0.0</k2>
+                    <k3>0.0</k3>
+                    <p1>0.0</p1>
+                    <p2>0.0</p2>
+                    <center>0.5 0.5</center>
+                </distortion>
+                <clip>
+                    <near>0.02</near>
+                    <far>30</far>
+                </clip>
+            </camera>
+            <plugin name="camera_controller" filename="libgazebo_ros_camera.so">
+                <alwaysOn>true</alwaysOn>
+                <updateRate>0.0</updateRate>
+                <cameraName>rgb_camera_sensor</cameraName>
+                <imageTopicName>/rgb_camera_sensor/image_raw</imageTopicName>
+                <cameraInfoTopicName>/rgb_camera_sensor/camera_info</cameraInfoTopicName>
+                <frameName>camera_link_optical</frameName>
+                <hackBaseline>0.0</hackBaseline>
+                <distortionK1>0.0</distortionK1>
+                <distortionK2>0.0</distortionK2>
+                <distortionK3>0.0</distortionK3>
+                <distortionT1>0.0</distortionT1>
+                <distortionT2>0.0</distortionT2>
+                <CxPrime>0</CxPrime>
+                <Cx>0.0</Cx>
+                <Cy>0.0</Cy>
+                <focalLength>0.0</focalLength>
+            </plugin>
+        </sensor>
+    </gazebo>
+    <joint name="rgb_camera_to_base_link" type="fixed">
+        <parent link="base_link" />
+        <child link="rgb_camera " />
+        <origin rpy="0 0 0" xyz="0 0 0" />
+    </joint>
     <link name="base_plate">
+        <xacro:default_inertial mass="0.1" />
         <visual>
             <origin rpy="0 0 0" xyz="-0.39 -0.39 -0.56" />
@@ -26,5 +114,13 @@
                     scale="0.01 0.01 0.01" />
             </geometry>
-        </visual>
+            <material name="red"/>
+        </visual>
+        <collision>
+            <origin rpy="0 0 0" xyz="-0.39 -0.39 -0.56" />
+            <geometry>
+                <mesh filename="package://arduinobot_description/meshes/base_plate.STL"
+                    scale="0.01 0.01 0.01" />
+            </geometry>
+        </collision>
     </link>
     <joint name="joint_1" type="revolute">
@@ -36,4 +132,5 @@
     </joint>
     <link name="forward_drive_arm">
+        <xacro:default_inertial mass="0.1" />
         <visual>
             <origin rpy="0 -${PI/2} ${PI/2}" xyz="0.19 0.06 -0.08" />
@@ -42,5 +139,13 @@
                     scale="0.01 0.01 0.01" />
             </geometry>
-        </visual>
+            <material name="orange"/>
+        </visual>
+        <collission>
+            <origin rpy="0 -${PI/2} ${PI/2}" xyz="0.19 0.06 -0.08" />
+            <geometry>
+                <mesh filename="package://arduinobot_description/meshes/forward_drive_arm.STL"
+                    scale="0.01 0.01 0.01" />
+            </geometry>
+        </collission>
     </link>
     <joint name="joint_2" type="revolute">
@@ -52,4 +157,5 @@
     </joint>
     <link name="horizontal_arm">
+        <xacro:default_inertial mass="0.1" />
         <visual>
             <origin rpy="${PI/2} 0 ${PI/2}" xyz="-0.03 -0.4 -0.06" />
@@ -58,5 +164,13 @@
                     scale="0.01 0.01 0.01" />
             </geometry>
-        </visual>
+            <material name="green"/>
+        </visual>
+        <collision>
+            <origin rpy="${PI/2} 0 ${PI/2}" xyz="-0.03 -0.4 -0.06" />
+            <geometry>
+                <mesh filename="package://arduinobot_description/meshes/horizontal_arm.STL"
+                    scale="0.01 0.01 0.01" />
+            </geometry>
+        </collision>
     </link>
     <joint name="joint_3" type="revolute">
@@ -68,4 +182,5 @@
     </joint>
     <link name="claw_support">
+        <xacro:default_inertial mass="0.05" />
         <visual>
             <origin rpy="0 0 ${PI/2}" xyz="0.13 -0.05 -0.15" />
@@ -74,5 +189,13 @@
                     scale="0.01 0.01 0.01" />
             </geometry>
-        </visual>
+            <material name="red"/>
+        </visual>
+        <collision>
+            <origin rpy="0 0 ${PI/2}" xyz="0.13 -0.05 -0.15" />
+            <geometry>
+                <mesh filename="package://arduinobot_description/meshes/claw_support.STL"
+                    scale="0.01 0.01 0.01" />
+            </geometry>
+        </collision>
     </link>
     <joint name="horizontal_arm_to_claw_support" type="fixed">
@@ -81,5 +204,29 @@
         <origin rpy="0 0 0" xyz="0 0.82 0" />
     </joint>
+    <link name="pi_camera ">
+        <xacro:default_inertial mass="0.01" />
+        <visual>
+            <origin rpy="${PI/3} ${PI} ${PI}" xyz="-0.12 0.26 0.31" />
+            <geometry>
+                <mesh filename="package://arduinobot_description/meshes/pi_camera.STL"
+                    scale="0.01 0.01 0.01" />
+            </geometry>
+            <material name="blue"/>
+        </visual>
+        <collision>
+            <origin rpy="${PI/3} ${PI} ${PI}" xyz="-0.12 0.26 0.31" />
+            <geometry>
+                <mesh filename="package://arduinobot_description/meshes/pi_camera.STL"
+                    scale="0.01 0.01 0.01" />
+            </geometry>
+        </collision>
+    </link>
+    <joint name="claw_support_to_pi_camera" type="fixed">
+        <parent link="claw_support" />
+        <child link="pi_camera " />
+        <origin rpy="0 0 0" xyz="0 0 0" />
+    </joint>
     <link name="gripper_right">
+        <xacro:default_inertial mass="0.01" />
         <visual>
             <origin rpy="0 0 -${PI/2}" xyz="-0.09 0.48 -0.08" />
@@ -88,7 +235,16 @@
                     scale="0.01 0.01 0.01" />
             </geometry>
-        </visual>
+            <material name="yellow"/>
+        </visual>
+        <collision>
+            <origin rpy="0 0 -${PI/2}" xyz="-0.09 0.48 -0.08" />
+            <geometry>
+                <mesh filename="package://arduinobot_description/meshes/right_finger.STL"
+                    scale="0.01 0.01 0.01" />
+            </geometry>
+        </collision>
     </link>
     <link name="gripper_left">
+        <xacro:default_inertial mass="0.01" />
         <visual>
             <origin rpy="0 0 -${PI/2}" xyz="-0.03 0.48 -0.08" />
@@ -97,5 +253,13 @@
                     scale="0.01 0.01 0.01" />
             </geometry>
-        </visual>
+            <material name="yellow"/>
+        </visual>
+        <collision>
+            <origin rpy="0 0 -${PI/2}" xyz="-0.03 0.48 -0.08" />
+            <geometry>
+                <mesh filename="package://arduinobot_description/meshes/left_finger.STL"
+                    scale="0.01 0.01 0.01" />
+            </geometry>
+        </collision>
     </link>
     <joint name="joint_4" type="revolute">
@@ -114,3 +278,30 @@
         <mimic joint="joint_4" multiplier="-1" />
     </joint>
+  <material name="black">
+    <color rgba="0.0 0.0 0.0 1.0"/>
+  </material>
+  <material name="blue">
+    <color rgba="0.0 0.0 0.8 1.0"/>
+  </material>
+  <material name="green">
+    <color rgba="0.0 0.8 0.0 1.0"/>
+  </material>
+  <material name="grey">
+    <color rgba="0.2 0.2 0.2 1.0"/>
+  </material>
+  <material name="orange">
+    <color rgba="${255/255} ${108/255} ${10/255} 1.0"/>
+  </material>
+  <material name="brown">
+    <color rgba="${222/255} ${207/255} ${195/255} 1.0"/>
+  </material>
+  <material name="red">
+    <color rgba="0.8 0.0 0.0 1.0"/>
+  </material>
+  <material name="white">
+    <color rgba="1.0 1.0 1.0 1.0"/>
+  </material>
+    <material name="yellow">
+    <color rgba="1.0 1.0 0.0 1.0"/>
+  </material>
 </robot>

Commit message: Controller setup

File: src/arduinobot_description/urdf/arduinobot.urdf.xacro (robot description, xacro)
@@ -1,4 +1,8 @@
 <?xml version="1.0"?>
 <robot xmlns:xacro="http://www.ros.org/wiki/xacro" name="arduinobot">
+    <xacro:arg name="is_ignition" default="false" />
+    <xacro:include filename="$(find arduinobot_description)/urdf/arduinobot_colors.xacro" />
+    <xacro:include filename="$(find arduinobot_description)/urdf/arduinobot_gazebo.xacro" />
+    <xacro:include filename="$(find arduinobot_description)/urdf/arduinobot_ros2_control.xacro" />
     <xacro:property name="PI" value="3.14159" />
     <xacro:property name="effort" value="30.0" />
@@ -21,5 +25,5 @@
                     scale="0.01 0.01 0.01" />
             </geometry>
-            <material name="red"/>
+            <material name="red" />
         </visual>
         <collision>
@@ -44,5 +48,5 @@
                     scale="0.01 0.01 0.01" />
             </geometry>
-            <material name="blue"/>
+            <material name="blue" />
         </visual>
         <collision>
@@ -114,5 +118,5 @@
                     scale="0.01 0.01 0.01" />
             </geometry>
-            <material name="red"/>
+            <material name="red" />
         </visual>
         <collision>
@@ -139,5 +143,5 @@
                     scale="0.01 0.01 0.01" />
             </geometry>
-            <material name="orange"/>
+            <material name="orange" />
         </visual>
         <collission>
@@ -164,5 +168,5 @@
                     scale="0.01 0.01 0.01" />
             </geometry>
-            <material name="green"/>
+            <material name="green" />
         </visual>
         <collision>
@@ -189,5 +193,5 @@
                     scale="0.01 0.01 0.01" />
             </geometry>
-            <material name="red"/>
+            <material name="red" />
         </visual>
         <collision>
@@ -212,5 +216,5 @@
                     scale="0.01 0.01 0.01" />
             </geometry>
-            <material name="blue"/>
+            <material name="blue" />
         </visual>
         <collision>
@@ -235,5 +239,5 @@
                     scale="0.01 0.01 0.01" />
             </geometry>
-            <material name="yellow"/>
+            <material name="yellow" />
         </visual>
         <collision>
@@ -253,5 +257,5 @@
                     scale="0.01 0.01 0.01" />
             </geometry>
-            <material name="yellow"/>
+            <material name="yellow" />
         </visual>
         <collision>
@@ -278,30 +282,3 @@
         <mimic joint="joint_4" multiplier="-1" />
     </joint>
-  <material name="black">
-    <color rgba="0.0 0.0 0.0 1.0"/>
-  </material>
-  <material name="blue">
-    <color rgba="0.0 0.0 0.8 1.0"/>
-  </material>
-  <material name="green">
-    <color rgba="0.0 0.8 0.0 1.0"/>
-  </material>
-  <material name="grey">
-    <color rgba="0.2 0.2 0.2 1.0"/>
-  </material>
-  <material name="orange">
-    <color rgba="${255/255} ${108/255} ${10/255} 1.0"/>
-  </material>
-  <material name="brown">
-    <color rgba="${222/255} ${207/255} ${195/255} 1.0"/>
-  </material>
-  <material name="red">
-    <color rgba="0.8 0.0 0.0 1.0"/>
-  </material>
-  <material name="white">
-    <color rgba="1.0 1.0 1.0 1.0"/>
-  </material>
-    <material name="yellow">
-    <color rgba="1.0 1.0 0.0 1.0"/>
-  </material>
 </robot>

Commit message: Working simulation

File: src/arduinobot_description/urdf/arduinobot.urdf.xacro (robot description, xacro)
@@ -40,8 +40,8 @@
         <origin rpy="0 0 0" xyz="0 0 0" />
     </joint>
-    <link name="rgb_camera ">
-        <xacro:default_inertial mass="0.01" />
-        <visual>
-            <origin rpy="${2*PI/3} ${PI} ${PI}" xyz="-0.127 0.35 0.3" />
+    <link name="rgb_camera">
+        <xacro:default_inertial mass="0.01" />
+        <visual>
+            <origin rpy="${2*PI/3} ${PI} ${PI}" xyz="-0.127 0.35 0.285" />
             <geometry>
                 <mesh filename="package://arduinobot_description/meshes/pi_camera.STL"
@@ -51,5 +51,5 @@
         </visual>
         <collision>
-            <origin rpy="${2*PI/3} ${PI} ${PI}" xyz="-0.127 0.35 0.3" />
+            <origin rpy="${2*PI/3} ${PI} ${PI}" xyz="-0.127 0.35 0.285" />
             <geometry>
                 <mesh filename="package://arduinobot_description/meshes/pi_camera.STL"
@@ -90,5 +90,5 @@
     <joint name="rgb_camera_to_base_link" type="fixed">
         <parent link="base_link" />
-        <child link="rgb_camera " />
+        <child link="rgb_camera" />
         <origin rpy="0 0 0" xyz="0 0 0" />
     </joint>
@@ -191,5 +191,5 @@
         <origin rpy="0 0 0" xyz="0 0.82 0" />
     </joint>
-    <link name="pi_camera ">
+    <link name="pi_camera">
         <xacro:default_inertial mass="0.01" />
         <visual>
@@ -211,5 +211,5 @@
     <joint name="claw_support_to_pi_camera" type="fixed">
         <parent link="claw_support" />
-        <child link="pi_camera " />
+        <child link="pi_camera" />
         <origin rpy="0 0 0" xyz="0 0 0" />
     </joint>

Commit message: robot-bringup

File: src/arduinobot_description/urdf/arduinobot.urdf.xacro (robot description, xacro)
@@ -1,5 +1,7 @@
 <?xml version="1.0"?>
 <robot xmlns:xacro="http://www.ros.org/wiki/xacro" name="arduinobot">
+    <xacro:arg name="port" default="/dev/ttyACM0" />
     <xacro:arg name="is_ignition" default="false" />
+    <xacro:arg name="is_sim" default="true" />
     <xacro:include filename="$(find arduinobot_description)/urdf/arduinobot_colors.xacro" />
     <xacro:include filename="$(find arduinobot_description)/urdf/arduinobot_gazebo.xacro" />

File: src/arduinobot_description/urdf/arduinobot_ros2_control.xacro (robot description, xacro)
@@ -3,14 +3,28 @@
     <xacro:property name="PI" value="3.14159" />
     <ros2_control type="system" name="RobotSystem">
-        <!-- ROS 2 Humble -->
-        <xacro:if value="$(arg is_ignition)">
+        <xacro:if value="$(arg is_sim)">
+            <!-- Simulation -->
+            <xacro:if value="$(arg is_ignition)">
+            <!-- ROS 2 Humble -->
+                <hardware>
+                    <plugin>ign_ros2_control/IgnitionSystem</plugin>
+                </hardware>
+            </xacro:if>
+            <xacro:unless value="$(arg is_ignition)">
+            <!-- ROS 2 Iron or above -->
+                <hardware>
+                    <plugin>gz_ros2_control/GazeboSimSystem</plugin>
+                </hardware>
+            </xacro:unless>
+            <joint name="joint_5">
+                <param name="mimic">joint_4</param>
+                <param name="multiplier">-1</param>
+            </joint>
+        </xacro:if>
+        <xacro:unless value="$(arg is_sim)">
+            <!-- Real Robot-->
             <hardware>
-                <plugin>ign_ros2_control/IgnitionSystem</plugin>
-            </hardware>
-        </xacro:if>
-        <!-- ROS 2 Iron or above -->
-        <xacro:unless value="$(arg is_ignition)">
-            <hardware>
-                <plugin>gz_ros2_control/GazeboSimSystem</plugin>
+                <plugin>arduinobot_controller/ArduinobotInterface</plugin>
+                <param name="port">$(arg port)</param>
             </hardware>
         </xacro:unless>
@@ -20,5 +34,5 @@
                 <param name="max">${PI/2}</param>
             </command_interface>
-            <state_interface name="position"/>
+            <state_interface name="position" />
         </joint>
         <joint name="joint_2">
@@ -27,5 +41,5 @@
                 <param name="max">${PI/2}</param>
             </command_interface>
-            <state_interface name="position"/>
+            <state_interface name="position" />
         </joint>
         <joint name="joint_3">
@@ -34,5 +48,5 @@
                 <param name="max">${PI/2}</param>
             </command_interface>
-            <state_interface name="position"/>
+            <state_interface name="position" />
         </joint>
         <joint name="joint_4">
@@ -41,9 +55,5 @@
                 <param name="max">0.0</param>
             </command_interface>
-            <state_interface name="position"/>
-        </joint>
-        <joint name="joint_5">
-            <param name="mimic">joint_4</param>
-            <param name="multiplier">-1</param>
+            <state_interface name="position" />
         </joint>
     </ros2_control>
