Commit message: Working robot (backwards)

File: src/arduinobot_description/urdf/arduinobot.urdf.xacro (robot description, xacro)
@@ -1,5 +1,5 @@
 <?xml version="1.0"?>
 <robot xmlns:xacro="http://www.ros.org/wiki/xacro" name="arduinobot">
-    <xacro:arg name="port" default="/dev/ttyACM0" />
+    <xacro:arg name="port" default="" />
     <xacro:arg name="is_ignition" default="false" />
     <xacro:arg name="is_sim" default="true" />
@@ -130,5 +130,5 @@
             <material name="orange" />
         </visual>
-        <collission>
+        <collision>
             <origin rpy="0 -${PI/2} ${PI/2}" xyz="0.19 0.06 -0.08" />
             <geometry>
@@ -136,5 +136,5 @@
                     scale="0.01 0.01 0.01" />
             </geometry>
-        </collission>
+        </collision>
     </link>
     <joint name="joint_2" type="revolute">
@@ -267,3 +267,17 @@
         <mimic joint="joint_4" multiplier="-1" />
     </joint>
+    <!-- Transmissions-->
+    <xacro:macro name="default_transmission" params="number">
+        <transmission name="transmission_${number}">
+            <plugin>transmission_interface/SimpleTransmission</plugin>
+            <actuator name="motor_${number}" role="actuator1"/>
+            <joint name="joint_${number}"    role="joint1">
+                <mechanical_reduction>1.0</mechanical_reduction>
+            </joint>
+        </transmission>
+    </xacro:macro>
+    <xacro:default_transmission number="1"/>
+    <xacro:default_transmission number="2"/>
+    <xacro:default_transmission number="3"/>
+    <xacro:default_transmission number="4"/>
 </robot>

File: src/arduinobot_description/urdf/arduinobot_ros2_control.xacro (robot description, xacro)
@@ -26,5 +26,5 @@
             <hardware>
                 <plugin>arduinobot_controller/ArduinobotInterface</plugin>
-                <param name="port">$(arg port)</param>
+                <param name="port">/dev/ttyACM0</param>
             </hardware>
         </xacro:unless>
